Commit message: robot urdf modification

File: urdf/robot.urdf (robot description, URDF)
Before this commit: robot robot_xacro, 7 links, 6 joints
Joints:
- joint hokuyo_joint: origin xyz=0.14 0 0.025 rpy=0 0 0 -> xyz=0.20 0 0.025 rpy=0 0 0
- joint neck_joint: origin xyz=0.20 0 0 rpy=0 0 0 -> xyz=0.13 0 0 rpy=0 0 0

File: urdf/robot.xacro (robot description, xacro)
@@ -1,5 +1,5 @@
 <?xml version="1.0"?>
 <robot xmlns:xacro="http://www.ros.org/wiki/xacro" name="robot_xacro">
-<xacro:include filename="$(find exp_assignment2)/urdf/robot.gazebo"/>
+<xacro:include filename="$(find exp_assignment3)/urdf/robot.gazebo"/>
 <!--	<xacro:macro name="cylinder_inertia" params="mass r l">
 	   <inertia ixx="${mass*(3*r*r+l*l)/12}" ixy = "0" ixz = "0"
@@ -188,5 +188,5 @@
   </joint>
   <joint name="neck_joint" type="fixed">
-  	<origin rpy="0 0 0" xyz="0.20 0 0"/>
+  	<origin rpy="0 0 0" xyz="0.13 0 0"/>
   	<parent link="link_chassis"/>
   	<child link="neck"/>
@@ -222,5 +222,5 @@
   <joint name="hokuyo_joint" type="fixed">
 	    <axis xyz="0 1 0" />
-	    <origin xyz="0.14 0 0.025" rpy="0 0 0"/>
+	    <origin xyz="0.20 0 0.025" rpy="0 0 0"/>
 	    <parent link="link_chassis"/>
 	    <child link="hokuyo_link"/>

Commit message: Improvement urdf robot

File: urdf/robot.urdf (robot description, URDF)
Before this commit: robot robot_xacro, 7 links, 6 joints
Joints:
- joint hokuyo_joint: origin xyz=0.20 0 0.025 rpy=0 0 0 -> xyz=0.26 0 0.025 rpy=0 0 0
- joint neck_joint: origin xyz=0.13 0 0 rpy=0 0 0 -> xyz=0.20 0 0 rpy=0 0 0

File: urdf/robot.xacro (robot description, xacro)
@@ -127,5 +127,5 @@
   	</inertial>
   	<collision>
-  	  <origin xyz="0 0 0.08" rpy="0 0 0"/>
+  	  <origin xyz="0 0 0.07" rpy="0 0 0"/>
       <geometry>
         <cylinder radius="0.04" length="0.08"/>
@@ -133,5 +133,5 @@
   	</collision>
   	<visual>
-  	  <origin xyz="0 0 0.08" rpy="0 0 0"/>
+  	  <origin xyz="0 0 0.07" rpy="0 0 0"/>
       <geometry>
         <cylinder radius="0.04" length="0.08"/>
@@ -143,9 +143,9 @@
   	<inertial>
 	<mass value="0.025"/>
-	<origin xyz="0 0 0.18" rpy="0 0 0" />
+	<origin xyz="0 0 0.15" rpy="0 0 0" />
 	<inertia ixx="0.000010279" ixy="0" ixz="0" iyy="0.000010279" iyz="0" izz="0.000007225"/>
   	</inertial>
   	<collision>
-  	  <origin xyz="0 0 0.18" rpy="0 0 0"/>
+  	  <origin xyz="0 0 0.16" rpy="0 0 0"/>
       <geometry>
         <box size="0.1 0.1 0.1"/>
@@ -153,5 +153,5 @@
   	</collision>
   	<visual>
-  	  <origin xyz="0 0 0.18" rpy="0 0 0"/>
+  	  <origin xyz="0 0 0.16" rpy="0 0 0"/>
       <geometry>
         <box size="0.1 0.1 0.1"/>
@@ -182,13 +182,13 @@
     </inertial>
   </link>
+  <joint name="neck_joint" type="fixed">
+  	<origin rpy="0 0 0" xyz="0.20 0 0"/>
+  	<parent link="link_chassis"/>
+  	<child link="neck"/>
+  </joint>
   <joint name="head_joint" type="fixed">
   	<origin rpy="0 0 0" xyz="0 0 0"/>
   	<parent link="neck"/>
   	<child link="head"/>
-  </joint>
-  <joint name="neck_joint" type="fixed">
-  	<origin rpy="0 0 0" xyz="0.13 0 0"/>
-  	<parent link="link_chassis"/>
-  	<child link="neck"/>
   </joint>
   <joint name="camera_joint" type="fixed">
@@ -222,5 +222,5 @@
   <joint name="hokuyo_joint" type="fixed">
 	    <axis xyz="0 1 0" />
-	    <origin xyz="0.20 0 0.025" rpy="0 0 0"/>
+	    <origin xyz="0.26 0 0.025" rpy="0 0 0"/>
 	    <parent link="link_chassis"/>
 	    <child link="hokuyo_link"/>
